File: kicad-projects/pmod-microsd-socket/pmod-microsd-socket.kicad_sch (KiCad schematic)
At the start: 2 parts, among them J1 PMOD_Peripheral_Conn_02x06, J2 Micro_SD_Card

Commit message: wip: board schematic and simulation
Parts:
- removed J1: PMOD_Peripheral_Conn_02x06, pmod:PMOD_PinHeader_2x06_P2.54mm_Horizontal, symbol pmod:PMOD_Peripheral_Conn_02x06
- removed J2: Micro_SD_Card, symbol Connector:Micro_SD_Card
- added C1: 100n, Capacitor_SMD:C_0603_1608Metric, symbol Device:C_Small
- added J1: PMOD_Host_Conn_02x06, pmod:PMOD_PinSocket_2x06_P2.54mm_Horizontal, symbol pmod:PMOD_Host_Conn_02x06
- added J2: Detect Switch, Connector_PinHeader_2.54mm:PinHeader_1x02_P2.54mm_Vertical, symbol Connector_Generic:Conn_01x02
- added J3: Micro_SD_Card_Det2, Connector_Card:microSD_HC_Hirose_DM3D-SF, symbol Connector:Micro_SD_Card_Det2
- added R1: 0, Resistor_SMD:R_0603_1608Metric, symbol Device:R_Small
Connections:
- new net: J2.1 (Pin_1), J3.9 (DET_B)
- new net: J2.2 (Pin_2), J3.10 (DET_A)
- new net: J3.11 (SHIELD), R1.1
- new net CLK: J1.7 (B0), J3.5 (CLK)
- new net CMD: J1.3 (A2), J3.3 (CMD)
- new net DAT0: J1.4 (A3), J3.7 (DAT0)
- new net DAT1: J1.10 (B3), J3.8 (DAT1)
- new net DAT2: J1.1 (A0), J3.1 (DAT2)
- new net DAT3: J1.2 (A1), J3.2 (DAT3/CD)
- new net GND: C1.2, J1.11 (GND), J1.5 (GND), J3.6 (VSS), R1.2
- new net VCC: C1.1, J1.12 (VCC), J1.6 (VCC), J3.4 (VDD)
- no-connect marks 0 -> 2
Other:
- note added: "SD card decoupling"
- note added: "TODO: Add terminations?"
